File: pt100.kicad_sch (KiCad schematic)
At the start: 14 parts, among them J5 Conn_01x03_Socket, J6 Conn_01x03_Socket, U4 TLV9002S

Commit message: wip schematic
Changed lines of the file:
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@@
 	)
 	(hierarchical_label "PT100_1"
-		(shape bidirectional)
+		(shape output)
 		(at 96.52 38.1 0)
 		(effects
@@
 	)
 	(hierarchical_label "SHDN1"
-		(shape bidirectional)
+		(shape input)
 		(at 80.01 29.21 90)
 		(effects
@@
 	)
 	(hierarchical_label "SHDN2"
-		(shape bidirectional)
+		(shape input)
 		(at 80.01 74.93 90)
 		(effects
@@
 	)
 	(hierarchical_label "PT100_2"
-		(shape bidirectional)
+		(shape output)
 		(at 96.52 83.82 0)
 		(effects

Commit message: wip - schematic and layout
Connections:
- net +3.3V renamed +1.8V

Commit message: wip
lcsc part numbers
Parts:
- removed R12, R17: 33K, Resistor_SMD:R_0603_1608Metric, symbol Resistor_E12_0603:Resistor 33K
- added R12, R17, R25, R29: 1M .1%, Resistor_SMD:R_0603_1608Metric, symbol Resistor_E12_0603:Resistor 1M
- added R24, R26, R27, R28: 3K3 .1%, Resistor_SMD:R_0603_1608Metric, symbol Resistor_E12_0603:Resistor 3K3
- R10, R15: value 91R -> 91R .1%; LCSC (none) -> C862316
- R11, R13, R14, R9: value 10K -> 10K .1%; LCSC C25804 -> C95204
Connections:
- net +1.8V: now also R24.1, R26.1, R27.1, R28.1; no longer R11.1, R13.1, R14.1, R9.1
- net GND: now also J5.1 (Pin_1), J6.1 (Pin_1), R12.2, R29.2; no longer J5.3 (Pin_3), J6.3 (Pin_3)
- net PT100_1: now also R17.2
- net PT100_2: now also R25.2
- net at C11.1, J5.2 (Pin_2): now also R9.1; no longer U4.3 (+)
- net at R13.2: now also U4.8 (-), R25.1; no longer J6.1 (Pin_1)
- net at C12.1, J6.2 (Pin_2): now also R14.1; no longer U4.7 (+)
- net at R11.2: now also U4.2 (-), R17.1; no longer J5.1 (Pin_1)
- new net: R29.1, R9.2, U4.3 (+)
- new net: R10.1, R11.1, R28.2
- new net: R13.1, R15.1, R26.2
- new net: J6.3 (Pin_3), R24.2
- new net: R12.1, R14.2, U4.7 (+)
- new net: J5.3 (Pin_3), R27.2
Other:
- moved on the sheet: C11, C12, J5, J6, R10, R11, R13, R14, R15, R9
