File: Hardware/ESP32-C3_Dev.kicad_sch (KiCad schematic)
At the start: 0 parts

Commit message: license
Other:
- company: (none) -> hand-crafted-electronics
- title: (none) -> Overview
Changed lines of the file:
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@@
 	(generator_version "9.0")
 	(paper "A4")
+	(title_block
+		(title "Overview")
+		(date "2026-01-09")
+		(rev "2")
+		(company "hand-crafted-electronics")
+		(comment 1 "https://ohwr.org/cern_ohl_s_v2.txt")
+		(comment 2 "https://github.com/pellematrose/ESP32-C3_Sensor/")
+		(comment 3 "Licensed under CERN-OHL-S v2")
+		(comment 4 "2026 Per-Simon Saal")
+	)
 	(wire
 		(pts
