File: Hardware/ESP32-C3_Dev.kicad_sch (KiCad schematic)
At the start: 0 parts

Commit message: wip
custom design rule, optimized layout,
Other:
- sheet Controller ports: added PS; removed SHDNLDO
- sheet Power Supply ports: added PS; removed SHDNLDO
Changed lines of the file:
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@@
 			)
 		)
-		(pin "SHDNLDO" output
+		(pin "PS" input
 			(at 147.32 67.31 180)
 			(effects
@@
 			)
 		)
-		(pin "SHDNLDO" input
+		(pin "PS" input
 			(at 135.89 67.31 0)
 			(effects
