File: Hardware/controller.kicad_sch (KiCad schematic)
At the start: 24 parts, among them SW1 SW_MEC_5G, SW2 SW_MEC_5G, U1 ESP32-C3-WROOM-02, U5 OLED_SSD1306, U8 BMP388

Commit message: housing created
Parts:
- added TP6: TestPoint, TestPoint:TestPoint_Pad_D1.5mm, symbol Connector:TestPoint
Connections:
- net SHDNLDO: no longer names the net of U1.6 (IO7)
- net SHDNLDO: now also TP6.1
Changed lines of the file:
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@@
-		)
-	)
-	(hierarchical_label "SHDNLDO"
-		(shape output)
-		(at 199.39 87.63 180)
-		(effects
-			(font
-				(size 1.27 1.27)
-			)
-			(justify right)
 		)
 	)
@@
 					(unit 1)
 				)
+			)
+		)
+	)
+	(symbol
+		(lib_id "Connector:TestPoint")
+		(at 199.39 87.63 90)
+		(unit 1)
+		(exclude_from_sim no)
+		(in_bom no)
+		(on_board yes)
+		(dnp no)
+		(property "Reference" "TP6"
+			(at 192.786 87.122 90)
+			(effects
+				(font
+					(size 1.27 1.27)
+				)
+			)
+		)
+		(property "Value" "TestPoint"
+			(at 196.088 92.71 90)
+			(effects
+				(font
+					(size 1.27 1.27)
+				)
+				(hide yes)
+			)
+		)
+		(property "Footprint" "TestPoint:TestPoint_Pad_D1.5mm"
+			(at 199.39 82.55 0)
+			(effects
+				(font
+					(size 1.27 1.27)
+				)
+				(hide yes)
+			)
+		)
+		(property "Datasheet" "~"
+			(at 199.39 82.55 0)
+			(effects
+				(font
+					(size 1.27 1.27)
+				)
+				(hide yes)
+			)
+		)
+		(property "Description" "test point"
+			(at 199.39 87.63 0)
+			(effects
+				(font
+					(size 1.27 1.27)
+				)
+				(hide yes)
+			)
+		)
+		(property "Characteristics" ""
+			(at 199.39 87.63 0)
+			(effects
+				(font
+					(size 1.27 1.27)
+				)
+				(hide yes)
+			)
+		)
+		(property "LCSC" ""
+			(at 199.39 87.63 0)
+			(effects
+				(font
+					(size 1.27 1.27)
+				)
+				(hide yes)
+			)
+		)
+		(pin "1"
+		)
+		(instances
+			(project "ESP32-C3_Dev"
+				(path "/db6fe335-723a-49f3-91f7-1db51b82a15a/91c554b6-9438-44a2-99d9-22b509dc076e"
+					(reference "TP6")
+					(unit 1)
+				)

Commit message: license
Other:
- company: (none) -> hand-crafted-electronics
- title: (none) -> Controller
Changed lines of the file:
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@@
 	(generator_version "9.0")
 	(paper "A4")
+	(title_block
+		(title "Controller")
+		(date "2026-01-09")
+		(rev "2")
+		(company "hand-crafted-electronics")
+		(comment 1 "https://ohwr.org/cern_ohl_s_v2.txt")
+		(comment 2 "https://github.com/pellematrose/ESP32-C3_Sensor/")
+		(comment 3 "Licensed under CERN-OHL-S v2")
+		(comment 4 "2026 Per-Simon Saal")
+	)
 	(text "BMP388 Address:\n1110110 x76"
 		(exclude_from_sim no)
