File: Hardware/controller.kicad_sch (KiCad schematic)
At the start: 25 parts, among them SW1 SW_MEC_5G, SW2 SW_MEC_5G, U1 ESP32-C3-WROOM-02, U5 OLED_SSD1306, U8 BMP388

Commit message: wip
custom design rule, optimized layout,
Parts:
- removed TP6: TestPoint, TestPoint:TestPoint_Pad_D1.5mm, symbol Connector:TestPoint
Connections:
- net PS: now reaches U1.6 (IO7)
Changed lines of the file:
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@@
 	(wire
 		(pts
-			(xy 196.85 100.33) (xy 203.2 100.33)
+			(xy 199.39 100.33) (xy 203.2 100.33)
 		)
 		(stroke
@@
 	(wire
 		(pts
-			(xy 196.85 97.79) (xy 203.2 97.79)
+			(xy 199.39 97.79) (xy 203.2 97.79)
 		)
 		(stroke
@@
 	(hierarchical_label "USB+"
 		(shape bidirectional)
-		(at 196.85 100.33 180)
+		(at 199.39 100.33 180)
 		(effects
 			(font
@@
 		)
 	)
+	(hierarchical_label "PS"
+		(shape input)
+		(at 199.39 87.63 180)
+		(effects
+			(font
+				(size 1.27 1.27)
+			)
+			(justify right)
+		)
+	)
 	(hierarchical_label "CHARGING"
 		(shape input)
@@
 	(hierarchical_label "USB-"
 		(shape bidirectional)
-		(at 196.85 97.79 180)
+		(at 199.39 97.79 180)
 		(effects
 			(font
@@
 					(unit 1)
 				)
-			)
-		)
-	)
-	(symbol
-		(lib_id "Connector:TestPoint")
-		(at 199.39 87.63 90)
-		(unit 1)
-		(exclude_from_sim no)
-		(in_bom no)
-		(on_board yes)
-		(dnp no)
-		(property "Reference" "TP6"
-			(at 192.786 87.122 90)
-			(effects
-				(font
-					(size 1.27 1.27)
-				)
-			)
-		)
-		(property "Value" "TestPoint"
-			(at 196.088 92.71 90)
-			(effects
-				(font
-					(size 1.27 1.27)
-				)
-				(hide yes)
-			)
-		)
-		(property "Footprint" "TestPoint:TestPoint_Pad_D1.5mm"
-			(at 199.39 82.55 0)
-			(effects
-				(font
-					(size 1.27 1.27)
-				)
-				(hide yes)
-			)
-		)
-		(property "Datasheet" "~"
-			(at 199.39 82.55 0)
-			(effects
-				(font
-					(size 1.27 1.27)
-				)
-				(hide yes)
-			)
-		)
-		(property "Description" "test point"
-			(at 199.39 87.63 0)
-			(effects
-				(font
-					(size 1.27 1.27)
-				)
-				(hide yes)
-			)
-		)
-		(property "Characteristics" ""
-			(at 199.39 87.63 0)
-			(effects
-				(font
-					(size 1.27 1.27)
-				)
-				(hide yes)
-			)
-		)
-		(property "LCSC" ""
-			(at 199.39 87.63 0)
-			(effects
-				(font
-					(size 1.27 1.27)
-				)
-				(hide yes)
-			)
-		)
-		(pin "1"
-		)
-		(instances
-			(project "ESP32-C3_Dev"
-				(path "/db6fe335-723a-49f3-91f7-1db51b82a15a/91c554b6-9438-44a2-99d9-22b509dc076e"
-					(reference "TP6")
-					(unit 1)
-				)

Commit message: big cleanup, new structure
added production and source folder for better structure
Parts:
- C15, C16, C4, C5, C7, C8: symbol _PS_LIB:C_0603 -> project_library:C_0603
- D6: symbol _PS_LIB:LED -> project_library:LED
- R22, R23, R30, R31, R4, R5, R6: symbol _PS_LIB:R_0603 -> project_library:R_0603
- SW1, SW2: symbol _PS_LIB:SW_MEC_5G -> project_library:SW_MEC_5G
- TP1, TP2, TP3, TP4, TP5: symbol Connector:TestPoint -> project_library:TestPoint
- U1: symbol RF_Module:ESP32-C3-WROOM-02 -> project_library:ESP32-C3-WROOM-02
- U5: symbol _PS_LIB:OLED_SSD1306 -> project_library:OLED_SSD1306
- U8: symbol BMP388:BMP388 -> project_library:BMP388
Changed lines of the file:
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@@
 	)
 	(symbol
-		(lib_id "_PS_LIB:C_0603")
+		(lib_id "project_library:C_0603")
 		(at 176.53 69.85 0)
 		(unit 1)
@@
 	)
 	(symbol
-		(lib_id "power:GND")
+		(lib_id "project_library:GND")
 		(at 237.49 50.8 0)
 		(unit 1)
@@
 	)
 	(symbol
-		(lib_id "power:+3.3V")
+		(lib_id "project_library:+3.3V")
 		(at 218.44 35.56 0)
 		(unit 1)
@@
 	)
 	(symbol
-		(lib_id "Connector:TestPoint")
+		(lib_id "project_library:TestPoint")
 		(at 74.93 74.93 90)
 		(unit 1)
@@
 	)
 	(symbol
-		(lib_id "power:GND")
+		(lib_id "project_library:GND")
 		(at 176.53 73.66 0)
 		(unit 1)
@@
 	)
 	(symbol
-		(lib_id "power:+5V")
+		(lib_id "project_library:+5V")
 		(at 78.74 80.01 270)
 		(unit 1)
@@
 	)
 	(symbol
-		(lib_id "Connector:TestPoint")
+		(lib_id "project_library:TestPoint")
 		(at 199.39 80.01 90)
 		(unit 1)
@@
 	)
 	(symbol
-		(lib_id "power:GND")
+		(lib_id "project_library:GND")
 		(at 165.1 64.77 270)
 		(unit 1)
@@
 	)
 	(symbol
-		(lib_id "power:GND")
+		(lib_id "project_library:GND")
 		(at 86.36 125.73 0)
 		(unit 1)
@@
 	)
 	(symbol
-		(lib_id "power:GND")
+		(lib_id "project_library:GND")
 		(at 78.74 74.93 90)
 		(unit 1)
@@
 	)
 	(symbol
-		(lib_id "power:+3.3V")
+		(lib_id "project_library:+3.3V")
 		(at 49.53 106.68 0)
 		(unit 1)
@@
 	)
 	(symbol
-		(lib_id "_PS_LIB:OLED_SSD1306")
+		(lib_id "project_library:OLED_SSD1306")
 		(at 121.92 41.91 90)
 		(unit 1)
@@
 	)
 	(symbol
-		(lib_id "_PS_LIB:SW_MEC_5G")
+		(lib_id "project_library:SW_MEC_5G")
 		(at 158.75 92.71 0)
 		(unit 1)
@@
 	)
 	(symbol
-		(lib_id "power:+3.3V")
+		(lib_id "project_library:+3.3V")
 		(at 176.53 90.17 90)
 		(unit 1)
@@
 	)
 	(symbol
-		(lib_id "_PS_LIB:R_0603")
+		(lib_id "project_library:R_0603")
 		(at 264.16 58.42 180)
 		(unit 1)
@@
 	)
 	(symbol
-		(lib_id "power:+3.3V")
+		(lib_id "project_library:+3.3V")
 		(at 264.16 52.07 0)
 		(unit 1)
@@
 	)
 	(symbol
-		(lib_id "_PS_LIB:R_0603")
+		(lib_id "project_library:R_0603")
 		(at 198.12 57.15 180)
 		(unit 1)
@@
 	)
 	(symbol
-		(lib_id "_PS_LIB:C_0603")
+		(lib_id "project_library:C_0603")
 		(at 237.49 46.99 0)
 		(unit 1)
@@
 	)
 	(symbol
-		(lib_id "_PS_LIB:SW_MEC_5G")
+		(lib_id "project_library:SW_MEC_5G")
 		(at 170.18 64.77 0)
 		(unit 1)
@@
 	)
 	(symbol
-		(lib_id "_PS_LIB:R_0603")
+		(lib_id "project_library:R_0603")
 		(at 182.88 90.17 270)
 		(unit 1)
@@
 	)
 	(symbol
-		(lib_id "power:+3.3V")
+		(lib_id "project_library:+3.3V")
 		(at 110.49 48.26 180)
 		(unit 1)
@@
 	)
 	(symbol
-		(lib_id "Connector:TestPoint")
+		(lib_id "project_library:TestPoint")
 		(at 199.39 82.55 90)
 		(unit 1)
@@
 	)
 	(symbol
-		(lib_id "_PS_LIB:R_0603")
+		(lib_id "project_library:R_0603")
 		(at 135.89 88.9 180)
 		(unit 1)
@@
 	)
 	(symbol
-		(lib_id "_PS_LIB:C_0603")
+		(lib_id "project_library:C_0603")
 		(at 97.79 113.03 0)
 		(unit 1)
@@
 	)
 	(symbol
-		(lib_id "power:GND")
+		(lib_id "project_library:GND")
 		(at 165.1 101.6 0)
 		(unit 1)
@@
 	)
 	(symbol
-		(lib_id "power:GND")
+		(lib_id "project_library:GND")
 		(at 165.1 82.55 270)
 		(unit 1)
@@
 	)
 	(symbol
-		(lib_id "Connector:TestPoint")
+		(lib_id "project_library:TestPoint")
 		(at 74.93 80.01 90)
 		(unit 1)
@@
 	)
 	(symbol
-		(lib_id "_PS_LIB:C_0603")
+		(lib_id "project_library:C_0603")
 		(at 165.1 97.79 0)
 		(unit 1)
@@
 	)
 	(symbol
-		(lib_id "power:GND")
+		(lib_id "project_library:GND")
 		(at 153.67 92.71 270)
 		(unit 1)
@@
 	)
 	(symbol
-		(lib_id "power:GND")
+		(lib_id "project_library:GND")
 		(at 218.44 105.41 0)
 		(unit 1)
@@
 	)
 	(symbol
-		(lib_id "power:+3.3V")
+		(lib_id "project_library:+3.3V")
 		(at 198.12 50.8 0)
 		(unit 1)
@@
 	)
 	(symbol
-		(lib_id "power:GND")
+		(lib_id "project_library:GND")
 		(at 105.41 48.26 0)
 		(unit 1)
@@
 	)
 	(symbol
-		(lib_id "power:+3.3V")
+		(lib_id "project_library:+3.3V")
 		(at 254 52.07 0)
 		(unit 1)
@@
 	)
 	(symbol
-		(lib_id "_PS_LIB:R_0603")
+		(lib_id "project_library:R_0603")
 		(at 180.34 82.55 270)
 		(unit 1)
@@
 	)
 	(symbol
-		(lib_id "Connector:TestPoint")
+		(lib_id "project_library:TestPoint")
 		(at 74.93 77.47 90)
 		(unit 1)
@@
 	)
 	(symbol
-		(lib_id "_PS_LIB:LED")
+		(lib_id "project_library:LED")
 		(at 135.89 97.79 90)
 		(unit 1)
@@
 	)
 	(symbol
-		(lib_id "_PS_LIB:R_0603")
+		(lib_id "project_library:R_0603")
 		(at 254 58.42 180)
 		(unit 1)
@@
 	)
 	(symbol
-		(lib_id "RF_Module:ESP32-C3-WROOM-02")
+		(lib_id "project_library:ESP32-C3-WROOM-02")
 		(at 218.44 82.55 0)
 		(unit 1)
@@
 	)
 	(symbol
-		(lib_id "power:GND")
+		(lib_id "project_library:GND")
 		(at 50.8 124.46 0)
 		(unit 1)
@@
 	)
 	(symbol
-		(lib_id "_PS_LIB:C_0603")
+		(lib_id "project_library:C_0603")
 		(at 223.52 46.99 0)
 		(unit 1)
@@
 	)
 	(symbol
-		(lib_id "_PS_LIB:C_0603")
+		(lib_id "project_library:C_0603")
 		(at 86.36 113.03 0)
 		(unit 1)
@@
 	)
 	(symbol
-		(lib_id "power:+3.3V")
+		(lib_id "project_library:+3.3V")
 		(at 76.2 102.87 0)
 		(unit 1)
@@
 	)
 	(symbol
-		(lib_id "power:GND")
+		(lib_id "project_library:GND")
 		(at 135.89 101.6 0)
 		(unit 1)
@@
 	)
 	(symbol
-		(lib_id "_PS_LIB:R_0603")
+		(lib_id "project_library:R_0603")
 		(at 168.91 82.55 270)
 		(unit 1)
@@
 	)
 	(symbol
-		(lib_id "BMP388:BMP388")
+		(lib_id "project_library:BMP388")
 		(at 63.5 116.84 0)
 		(unit 1)
@@
 	)
 	(symbol
-		(lib_id "power:+3.3V")
+		(lib_id "project_library:+3.3V")
 		(at 78.74 77.47 270)
 		(unit 1)
@@
 	)
 	(symbol
-		(lib_id "power:GND")
+		(lib_id "project_library:GND")
 		(at 223.52 50.8 0)
 		(unit 1)
