File: Hardware/ESP32-C3_Dev.kicad_pcb (KiCad board)
At the start: 2 copper layers, 32.7 x 47.2 mm, 95 parts, among them J1 Conn_01x02_Socket, J2 Conn_01x02_Socket, J4 USB_C_Receptacle_USB2.0_16P, J8 Conn_01x02_Pin, Q1 Dual_NMOS_8205A, Q2 DMG2305UX, SW1 SW_MEC_5G, SW2 SW_MEC_5G, U1 ESP32-C3-WROOM-02, U2 RT6150A, U3 DW01A, U4 TLV9002S, U5 OLED_SSD1306, U6 TP4056, U8 BMP388

Commit message: wip
custom design rule, optimized layout,
Parts:
- removed TP6: TestPoint, TestPoint:TestPoint_Pad_D1.5mm
- removed kibuzzard-68E986B5: G***, kibuzzard-68E986B5
- added kibuzzard-696E7314: G***, kibuzzard-696E7314, F.Cu at (128.3, 88.9)
- R35: moved to B.Cu
- moved C3 9.32 mm to (128.0, 94.5), turned to 90 degrees
- moved TP4 5.70 mm to (128.5, 91.3)
- moved C13 5.31 mm to (137.0, 94.3), turned to 90 degrees
- moved C18 5.05 mm to (129.7, 94.5), turned to 90 degrees
- moved D5 5.00 mm to (140.8, 84.5)
- moved R3 5.00 mm to (137.5, 84.5)
- moved L1 4.68 mm to (134.0, 97.3), turned to 180 degrees
- moved C8 4.61 mm to (131.5, 99.3), turned to -90 degrees
- moved R34 3.53 mm to (131.5, 92.3), turned to 90 degrees
- moved R33 3.02 mm to (131.5, 95.3), turned to 90 degrees
- moved U2 1.12 mm to (134.0, 94.3), turned to 90 degrees
- moved C9 1.00 mm to (142.2, 88.8)
- moved Q1 1.00 mm to (149.2, 89.0)
- moved R20 1.00 mm to (146.1, 86.5)
- moved R21 1.00 mm to (149.2, 86.5)
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Connections:
- U1 pad 6: Net-(U1-IO7) -> /Controller/PS
- U2 pad 7: /Power Supply/PS -> /Controller/PS
Routing:
- net /Controller/PS: track 0.00 -> 29.6 mm, vias 0 -> 2
- net +3.3V: track 153.5 -> 135.8 mm, vias 7 -> 4
- net /Controller/SHDN1: track 26.4 -> 21.2 mm
- net /Controller/EN: track 42.5 -> 45.5 mm
- net GND: track 35.5 -> 33.4 mm, vias 39 -> 36
- net Net-(J1-Pin_2): track 8.85 -> 10.9 mm
- net /Controller/PT100_1: track 34.5 -> 32.7 mm
- net +5V: track 34.4 -> 33.2 mm, vias 4 -> 5
- net /Power Supply/PS: track 1.05 -> 0.00 mm, vias 1 -> 0
- net /Power Supply/battery+: track 26.3 -> 27.3 mm
- net /Power Supply/battery-: track 14.4 -> 15.4 mm
- net Net-(U1-IO4): track 5.79 -> 6.45 mm
- net /Controller/UBAT: track 27.1 -> 27.8 mm
- net USB5V: track 42.6 -> 43.2 mm

Commit message: V2.1 finished and ordered
Parts:
- removed kibuzzard-6930773F: G***, kibuzzard-6930773F
- added H*: Stencil hole, _PS_LIB_PCB:Stencil hole, F.Cu at (127.0, 54.3)
- added H*: Stencil hole, _PS_LIB_PCB:Stencil hole, F.Cu at (155.0, 54.3)
- added REF**: Mouse_bite, _PS_LIB_PCB:Mouse_bite, F.Cu at (141.0, 58.6)
- added kibuzzard-69738792: G***, kibuzzard-69738792, B.Cu at (140.5, 101.0)
- moved D5 0.16 mm to (141.0, 84.5)
- moved J4 0.16 mm to (141.0, 102.1)
- moved R3 0.16 mm to (137.7, 84.5)
- moved U5 0.16 mm to (140.8, 87.0)
Routing:
- net USB5V: track 43.2 -> 42.5 mm
Other:
- board size 32.7 x 47.2 mm -> 33 x 54.2 mm
