File: Hardware/powersupply.kicad_sch (KiCad schematic)
At the start: 30 parts, among them J4 USB_C_Receptacle_USB2.0_16P, J8 Conn_01x02_Pin, Q1 Dual_NMOS_8205A, Q2 DMG2305UX, U2 RT6150A, U3 DW01A, U6 TP4056

Commit message: wip
Parts:
- removed L1: 2u2, Inductor_SMD:L_0603_1608Metric, symbol Device:L_Small
- added L1: 2u2 1A, _PS_LIB_PCB:Inductor_1210, symbol _PS_LIB:Inductor 2u2
Connections:
- net at U2.4 (LX1): now also L1.1
- net at U2.2 (LX2): now also L1.2

Commit message: big cleanup, new structure
added production and source folder for better structure
Parts:
- C13, C18: symbol _PS_LIB:C_1206 -> project_library:C_1206
- C17, C3, C6, C9: symbol _PS_LIB:C_0603 -> project_library:C_0603
- D1, D3, D4: symbol Diode:ESD5Zxx -> project_library:ESD5Zxx
- D2: symbol Diode:1N5819WS -> project_library:1N5819WS
- D5: symbol _PS_LIB:LED -> project_library:LED
- J4: symbol Connector:USB_C_Receptacle_USB2.0_16P -> project_library:USB_C_Receptacle_USB2.0_16P
- J8: symbol Connector:Conn_01x02_Pin -> project_library:Conn_01x02_Pin
- L1: symbol _PS_LIB:Inductor 2u2 -> project_library:Inductor 2u2
- Q1: symbol _PS_LIB:Dual_NMOS_8205A -> project_library:Dual_NMOS_8205A
- Q2: symbol Transistor_FET:Q_PMOS_GSD -> project_library:Q_PMOS_GSD
- R1, R2, R3: symbol _PS_LIB:R_0603 -> project_library:R_0603
- R16: symbol Resistor_E12_0603:Resistor 3K9 -> project_library:Resistor 3K9
- R20, R21: symbol Resistor_E12_0603:Resistor 100K -> project_library:Resistor 100K
- R32: symbol Resistor_E12_0603:Resistor 10K -> project_library:Resistor 10K
- R33: symbol Resistor_E12_0603:Resistor 470K -> project_library:Resistor 470K
- R34: symbol Resistor_E12_0603:Resistor 82K -> project_library:Resistor 82K
- R7: symbol Resistor_E12_0603:Resistor 100R -> project_library:Resistor 100R
- R8: symbol Resistor_E12_0603:Resistor 1K -> project_library:Resistor 1K
- U2: symbol PS_IC:RT6150A -> project_library:RT6150A
- U3: symbol Battery_Management:DW01A -> project_library:DW01A
- U6: symbol Battery_Management:TP4056-42-ESOP8 -> project_library:TP4056-42-ESOP8
Changed lines of the file:
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@@
 	)
 	(symbol
-		(lib_id "power:GND")
+		(lib_id "project_library:GND")
 		(at 190.5 45.72 0)
 		(unit 1)
@@
 	)
 	(symbol
-		(lib_id "power:+5V")
+		(lib_id "project_library:+5V")
 		(at 95.25 35.56 0)
 		(unit 1)
@@
 	)
 	(symbol
-		(lib_id "Resistor_E12_0603:Resistor 82K")
+		(lib_id "project_library:Resistor 82K")
 		(at 154.94 53.34 0)
 		(unit 1)
@@
 	)
 	(symbol
-		(lib_id "_PS_LIB:C_0603")
+		(lib_id "project_library:C_0603")
 		(at 144.78 135.89 0)
 		(mirror y)
@@
 	)
 	(symbol
-		(lib_id "_PS_LIB:Dual_NMOS_8205A")
+		(lib_id "project_library:Dual_NMOS_8205A")
 		(at 121.92 152.4 270)
 		(unit 2)
@@
 	)
 	(symbol
-		(lib_id "power:+5V")
+		(lib_id "project_library:+5V")
 		(at 86.36 102.87 0)
 		(unit 1)
@@
 	)
 	(symbol
-		(lib_id "Connector:USB_C_Receptacle_USB2.0_16P")
+		(lib_id "project_library:USB_C_Receptacle_USB2.0_16P")
 		(at 39.37 53.34 0)
 		(unit 1)
@@
 	)
 	(symbol
-		(lib_id "_PS_LIB:C_0603")
+		(lib_id "project_library:C_0603")
 		(at 86.36 144.78 0)
 		(unit 1)
@@
 	)
 	(symbol
-		(lib_id "power:GND")
+		(lib_id "project_library:GND")
 		(at 86.36 156.21 0)
 		(mirror y)
@@
 	)
 	(symbol
-		(lib_id "_PS_LIB:C_1206")
+		(lib_id "project_library:C_1206")
 		(at 165.1 41.91 0)
 		(unit 1)
@@
 	)
 	(symbol
-		(lib_id "power:GND")
+		(lib_id "project_library:GND")
 		(at 97.79 156.21 0)
 		(mirror y)
@@
 	)
 	(symbol
-		(lib_id "Battery_Management:TP4056-42-ESOP8")
+		(lib_id "project_library:TP4056-42-ESOP8")
 		(at 63.5 142.24 0)
 		(unit 1)
@@
 	)
 	(symbol
-		(lib_id "_PS_LIB:Dual_NMOS_8205A")
+		(lib_id "project_library:Dual_NMOS_8205A")
 		(at 135.89 152.4 90)
 		(mirror x)
@@
 	)
 	(symbol
-		(lib_id "power:GND")
+		(lib_id "project_library:GND")
 		(at 113.03 156.21 0)
 		(unit 1)
@@
 	)
 	(symbol
-		(lib_id "power:GND")
+		(lib_id "project_library:GND")
 		(at 77.47 45.72 90)
 		(unit 1)
@@
 	)
 	(symbol
-		(lib_id "power:GND")
+		(lib_id "project_library:GND")
 		(at 102.87 69.85 0)
 		(unit 1)
@@
 	)
 	(symbol
-		(lib_id "power:GND")
+		(lib_id "project_library:GND")
 		(at 180.34 45.72 0)
 		(unit 1)
@@
 	)
 	(symbol
-		(lib_id "power:GND")
+		(lib_id "project_library:GND")
 		(at 140.97 55.88 0)
 		(unit 1)
@@
 	)
 	(symbol
-		(lib_id "Resistor_E12_0603:Resistor 10K")
+		(lib_id "project_library:Resistor 10K")
 		(at 77.47 125.73 0)
 		(unit 1)
@@
 	)
 	(symbol
-		(lib_id "power:+5V")
+		(lib_id "project_library:+5V")
 		(at 115.57 35.56 0)
 		(unit 1)
@@
 	)
 	(symbol
-		(lib_id "Connector:Conn_01x02_Pin")
+		(lib_id "project_library:Conn_01x02_Pin")
 		(at 180.34 133.35 180)
 		(unit 1)
@@
 	)
 	(symbol
-		(lib_id "power:+5V")
+		(lib_id "project_library:+5V")
 		(at 44.45 157.48 0)
 		(unit 1)
@@
 	)
 	(symbol
-		(lib_id "_PS_LIB:C_0603")
+		(lib_id "project_library:C_0603")
 		(at 180.34 41.91 0)
 		(unit 1)
@@
 	)
 	(symbol
-		(lib_id "power:GND")
+		(lib_id "project_library:GND")
 		(at 80.01 69.85 0)
 		(unit 1)
@@
 	)
 	(symbol
-		(lib_id "power:GND")
+		(lib_id "project_library:GND")
 		(at 165.1 45.72 0)
 		(unit 1)
@@
 	)
 	(symbol
-		(lib_id "Diode:1N5819WS")
+		(lib_id "project_library:1N5819WS")
 		(at 107.95 38.1 180)
 		(unit 1)
@@
 	)
 	(symbol
-		(lib_id "power:GND")
+		(lib_id "project_library:GND")
 		(at 60.96 156.21 0)
 		(unit 1)
@@
 	)
 	(symbol
-		(lib_id "power:GND")
+		(lib_id "project_library:GND")
 		(at 31.75 76.2 0)
 		(unit 1)
@@
 	)
 	(symbol
-		(lib_id "Diode:ESD5Zxx")
+		(lib_id "project_library:ESD5Zxx")
 		(at 80.01 66.04 270)
 		(unit 1)
@@
 	)
 	(symbol
-		(lib_id "_PS_LIB:R_0603")
+		(lib_id "project_library:R_0603")
 		(at 71.12 45.72 90)
 		(unit 1)
@@
 	)
 	(symbol
-		(lib_id "_PS_LIB:R_0603")
+		(lib_id "project_library:R_0603")
 		(at 71.12 43.18 90)
 		(unit 1)
@@
 	)
 	(symbol
-		(lib_id "Battery_Management:DW01A")
+		(lib_id "project_library:DW01A")
 		(at 128.27 133.35 0)
 		(mirror y)
@@
 	)
 	(symbol
-		(lib_id "power:GND")
+		(lib_id "project_library:GND")
 		(at 135.89 55.88 0)
 		(unit 1)
@@
 	)
 	(symbol
-		(lib_id "Resistor_E12_0603:Resistor 100R")
+		(lib_id "project_library:Resistor 100R")
 		(at 152.4 130.81 270)
 		(mirror x)
@@
 	)
 	(symbol
-		(lib_id "power:GND")
+		(lib_id "project_library:GND")
 		(at 59.69 69.85 0)
 		(unit 1)
@@
 	)
 	(symbol
-		(lib_id "Transistor_FET:Q_PMOS_GSD")
+		(lib_id "project_library:Q_PMOS_GSD")
 		(at 83.82 119.38 0)
 		(mirror x)
@@
 	)
 	(symbol
-		(lib_id "Resistor_E12_0603:Resistor 1K")
+		(lib_id "project_library:Resistor 1K")
 		(at 113.03 142.24 0)
 		(mirror y)
@@
 	)
 	(symbol
-		(lib_id "_PS_LIB:R_0603")
+		(lib_id "project_library:R_0603")
 		(at 185.42 36.83 90)
 		(unit 1)
@@
 	)
 	(symbol
-		(lib_id "_PS_LIB:LED")
+		(lib_id "project_library:LED")
 		(at 190.5 41.91 90)
 		(unit 1)
@@
 	)
 	(symbol
-		(lib_id "power:+5V")
+		(lib_id "project_library:+5V")
 		(at 63.5 115.57 0)
 		(unit 1)
@@
 	)
 	(symbol
-		(lib_id "Diode:ESD5Zxx")
+		(lib_id "project_library:ESD5Zxx")
 		(at 102.87 60.96 270)
 		(unit 1)
@@
 	)
 	(symbol
-		(lib_id "_PS_LIB:Inductor 2u2")
+		(lib_id "project_library:Inductor 2u2")
 		(at 138.43 27.94 90)
 		(unit 1)
@@
 	)
 	(symbol
-		(lib_id "power:GND")
+		(lib_id "project_library:GND")
 		(at 44.45 165.1 0)
 		(unit 1)
@@
 	)
 	(symbol
-		(lib_id "Resistor_E12_0603:Resistor 100K")
+		(lib_id "project_library:Resistor 100K")
 		(at 97.79 152.4 0)
 		(unit 1)
@@
 	)
 	(symbol
-		(lib_id "power:GND")
+		(lib_id "project_library:GND")
 		(at 77.47 43.18 90)
 		(unit 1)
@@
 	)
 	(symbol
-		(lib_id "_PS_LIB:C_0603")
+		(lib_id "project_library:C_0603")
 		(at 44.45 161.29 0)
 		(mirror y)
@@
 	)
 	(symbol
-		(lib_id "power:GND")
+		(lib_id "project_library:GND")
 		(at 115.57 48.26 0)
 		(unit 1)
@@
 	)
 	(symbol
-		(lib_id "power:GND")
+		(lib_id "project_library:GND")
 		(at 63.5 156.21 0)
 		(unit 1)
@@
 	)
 	(symbol
-		(lib_id "power:GND")
+		(lib_id "project_library:GND")
 		(at 39.37 76.2 0)
 		(unit 1)
@@
 	)
 	(symbol
-		(lib_id "Resistor_E12_0603:Resistor 3K9")
+		(lib_id "project_library:Resistor 3K9")
 		(at 77.47 152.4 0)
 		(unit 1)
@@
 	)
 	(symbol
-		(lib_id "_PS_LIB:C_1206")
+		(lib_id "project_library:C_1206")
 		(at 115.57 44.45 0)
 		(unit 1)
@@
 	)
 	(symbol
-		(lib_id "Resistor_E12_0603:Resistor 100K")
+		(lib_id "project_library:Resistor 100K")
 		(at 97.79 142.24 0)
 		(unit 1)
@@
 	)
 	(symbol
-		(lib_id "Resistor_E12_0603:Resistor 470K")
+		(lib_id "project_library:Resistor 470K")
 		(at 154.94 41.91 0)
 		(unit 1)
@@
 	)
 	(symbol
-		(lib_id "power:GND")
+		(lib_id "project_library:GND")
 		(at 77.47 129.54 0)
 		(mirror y)
@@
 	)
 	(symbol
-		(lib_id "Diode:ESD5Zxx")
+		(lib_id "project_library:ESD5Zxx")
 		(at 59.69 66.04 270)
 		(unit 1)
@@
 	)
 	(symbol
-		(lib_id "power:GND")
+		(lib_id "project_library:GND")
 		(at 154.94 57.15 0)
 		(unit 1)
@@
 	)
 	(symbol
-		(lib_id "PS_IC:RT6150A")
+		(lib_id "project_library:RT6150A")
 		(at 138.43 41.91 0)
 		(unit 1)
@@
 	)
 	(symbol
-		(lib_id "power:GND")
+		(lib_id "project_library:GND")
 		(at 77.47 156.21 0)
 		(mirror y)
@@
 	)
 	(symbol
-		(lib_id "power:GND")
+		(lib_id "project_library:GND")
 		(at 138.43 55.88 0)
 		(unit 1)
@@
 	)
 	(symbol
-		(lib_id "power:+3.3V")
+		(lib_id "project_library:+3.3V")
 		(at 180.34 34.29 0)
 		(unit 1)
