File: Hardware/build/source/ESP32-C3_Dev.kicad_pcb (KiCad board)
At the start: 2 copper layers, 33 x 54.2 mm, 96 parts, among them J1 Conn_01x02_Socket, J2 Conn_01x02_Socket, J4 USB_C_Receptacle_USB2.0_16P, J8 Conn_01x02_Pin, Q1 Dual_NMOS_8205A, Q2 DMG2305UX, SW1 SW_MEC_5G, SW2 SW_MEC_5G, U1 ESP32-C3-WROOM-02, U2 RT6150A, U3 DW01A, U4 TLV9002S, U5 OLED_SSD1306, U6 TP4056, U8 BMP388

Commit message: wip
Parts:
- C1, C10, C11, C12, C15, C16, C17, C2, C3, C4, C5, C6, C7, C8, C9: footprint footprints_library:C_0603_1608Metric -> Capacitor_SMD:C_0603_1608Metric
- C13, C18: footprint footprints_library:C_0805_2012Metric -> Capacitor_SMD:C_0805_2012Metric
- D1, D3, D4: footprint footprints_library:D_SOD-523 -> Diode_SMD:D_SOD-523
- D2: footprint footprints_library:D_SOD-323 -> Diode_SMD:D_SOD-323
- D5, D6: footprint footprints_library:LED_0603_1608Metric -> LED_SMD:LED_0603_1608Metric
- J4: footprint footprints_library:USB_C_Receptacle_GCT_USB4105-xx-A_16P_TopMnt_Horizontal -> Connector_USB:USB_C_Receptacle_GCT_USB4105-xx-A_16P_TopMnt_Horizontal
- J8: footprint footprints_library:JST_PH_B2B-PH-K_1x02_P2.00mm_Vertical -> Connector_JST:JST_PH_B2B-PH-K_1x02_P2.00mm_Vertical
- L1: footprint footprints_library:Inductor_1210 -> _PS_LIB_PCB:Inductor_1210
- Q1, U3: footprint footprints_library:SOT-23-6 -> Package_TO_SOT_SMD:SOT-23-6
- Q2: footprint footprints_library:SOT-23-3 -> Package_TO_SOT_SMD:SOT-23-3
- R1, R10, R11, R12, R13, R14, R15, R16, R17, R2, R20, R21, R22, R23, R24, R25, R26, R27, R28, R29, R3, R30, R31, R32, R33, R34, R4, R5, R6, R7, R8, R9: footprint footprints_library:R_0603_1608Metric -> Resistor_SMD:R_0603_1608Metric
- R35: footprint footprints_library:R_0805_2012Metric -> Resistor_SMD:R_0805_2012Metric
- SW1, SW2: footprint footprints_library:Xunpu TS-1088 -> _PS_LIB_PCB:Xunpu TS-1088
- TP1, TP2, TP3, TP4, TP5: footprint footprints_library:TestPoint_Pad_D1.5mm -> TestPoint:TestPoint_Pad_D1.5mm
- U1: footprint footprints_library:ESP32-C3-WROOM-02 -> RF_Module:ESP32-C3-WROOM-02
- U2: footprint footprints_library:WDFN-10-1EP_3x3mm_P0.5mm_EP1.8x2.5mm -> Package_DFN_QFN:WDFN-10-1EP_3x3mm_P0.5mm_EP1.8x2.5mm
- U4: footprint footprints_library:VSSOP-10_3x3mm_P0.5mm -> Package_SO:VSSOP-10_3x3mm_P0.5mm
- U5: footprint footprints_library:SSD1306_0.96_Oled -> _PS_LIB_PCB:SSD1306_0.96_Oled
- U6: footprint footprints_library:SOIC-8-1EP_3.9x4.9mm_P1.27mm_EP2.41x3.3mm_ThermalVias -> Package_SO:SOIC-8-1EP_3.9x4.9mm_P1.27mm_EP2.41x3.3mm_ThermalVias
